File: Motor_Driver.kicad_pcb (KiCad board)
At the start: 2 copper layers, 61 x 31.1 mm, 42 parts, among them J1 Conn_01x04_Male, J2 Conn_01x40_Male, J3 Conn_01x02_Female, Q1 Q_NMOS_SGD, Q2 Q_NMOS_SGD, Q3 Q_NMOS_SGD, Q4 Q_NMOS_SGD, U1 NJM7812, U2 Si8274(DFN-14), U3 Si8274(DFN-14)

Commit message: 0.1 first
Parts:
- U2, U3: value Si8274(DFN-14) -> Si8274(SOIC-16); footprint Package_DFN_QFN_additional:DFN-14_4.9x4.9mm_P0.65mm -> Package_SO:SOIC-16_3.9x9.9mm_P1.27mm
- moved U3 0.35 mm to (149.9, 106.7)
- moved U2 0.29 mm to (149.9, 95.2)
Connections:
- U2 pad 1: Net-(U2-Pad1) -> PWM1
- U2 pad 10: +12V -> Low_1
- U2 pad 11: Net-(U2-Pad11) -> +12V
- U2 pad 12: Out_1 -> Net-(U2-Pad12)
- U2 pad 13: Hi_1 -> Net-(U2-Pad13)
- U2 pad 14: VB_1 -> Out_1
- U2 pad 2: PWM1 -> Net-(U2-Pad2)
- U2 pad 3: Net-(U2-Pad3) -> +3V3
- U2 pad 7: +3V3 -> Net-(U2-Pad7)
- U2 pad 8: GNDPWR -> +3V3
- U2 pad 9: Low_1 -> GNDPWR
- U3 pad 1: Net-(U3-Pad1) -> PWM2
- U3 pad 10: +12V -> Low_2
- U3 pad 11: Net-(U3-Pad11) -> +12V
- U3 pad 12: Out_2 -> Net-(U3-Pad12)
- U3 pad 13: Hi_2 -> Net-(U3-Pad13)
- U3 pad 14: VB_2 -> Out_2
- U3 pad 2: PWM2 -> Net-(U3-Pad2)
- U3 pad 3: Net-(U3-Pad3) -> +3V3
- U3 pad 7: +3V3 -> Net-(U3-Pad7)
- U3 pad 8: GNDPWR -> +3V3
- U3 pad 9: Low_2 -> GNDPWR
Routing:
- net +3V3: track 37.4 -> 47.6 mm
- net Out_2: track 36.2 -> 38.7 mm
- net Out_1: track 40.2 -> 38.5 mm
- net Hi_2: track 15.7 -> 14.5 mm
- net VB_2: track 8.69 -> 7.57 mm
- net PWM1: track 31.2 -> 30.1 mm
- net Net-(R4-Pad1): track 5.42 -> 4.51 mm
- net Hi_1: track 15.4 -> 14.5 mm
- net VB_1: track 8.46 -> 7.57 mm
- net Net-(R3-Pad1): track 5.38 -> 4.51 mm
- net +12V: track 56.8 -> 57.5 mm
- net Low_2: track 10.8 -> 10.1 mm
- net Low_1: track 12.8 -> 13.5 mm
- net GNDPWR: vias 41 -> 43
- net GND: vias 16 -> 12
Other:
- board text added: "MD-DI-1_0.1"
- board text removed: "MD-DI-1_1.0"
